Commit message: Update configs for simulations

File: src/na_launch/urdf/boat.urdf (robot description, URDF)
Before this commit: robot na_boat, 2 links, 1 joints
Links:
- removed link hull_marker
- link base_link: mass 70.0 -> None; geometry visual box size=0.15 0.15 0.15; visual box size=1.2 1.0 0.6
Joints:
- removed joint hull_fixed
